File: Hardware/MatrixDisplay.sch (KiCad schematic (older format))
At the start: 12 parts, among them U1 MAX7219, U2 MAX7219, U3 MAX7219, U4 MAX7219, U5 MAX7219, U6 MAX7219

Commit message: Create PCB and schematic
Parts:
- added C1, C2, C3, C4, C5, C6: 100n, Capacitors_SMD:C_0603_HandSoldering, symbol C_Small
- added LED1, LED2, LED3, LED4, LED5, LED6: 1088BS, LED_matrix:1088BS, symbol 1088BS
- added P1, P2, P3, P4: CONN_01X02, Connectors:socket_strip_smd_1x02, symbol CONN_01X02
- added P10, P11, P12, P9: CONN_01X04, Socket_Strips:Socket_Strip_Straight_1x04, symbol CONN_01X04
- added P5, P6, P7, P8: CONN_01X04, Connectors:socket_strip_smd_1x04, symbol CONN_01X04
- R1, R2, R3, R4, R5, R6: value R -> 10k; footprint (none) -> Resistors_SMD:R_0603_HandSoldering
- U1, U2, U3, U4, U5, U6: footprint (none) -> SMD_Packages:SOIC-24
Connections:
- net C11: now also LED1.4 (C1)
- net C12: now also LED1.14 (C2)
- net C13: now also LED1.13 (C3)
- net C14: now also LED1.7 (C4)
- net C15: now also LED1.11 (C5)
- net C16: now also LED1.6 (C6)
- net C17: now also LED1.2 (C7)
- net C18: now also LED1.1 (C8)
- net C21: now also LED4.4 (C1)
- net C22: now also LED4.14 (C2)
- net C23: now also LED4.13 (C3)
- net C24: now also LED4.7 (C4)
- net C25: now also LED4.11 (C5)
- net C26: now also LED4.6 (C6)
- net C27: now also LED4.2 (C7)
- net C28: now also LED4.1 (C8)
- net C31: now also LED2.4 (C1)
- net C32: now also LED2.14 (C2)
- net C33: now also LED2.13 (C3)
- net C34: now also LED2.7 (C4)
- net C35: now also LED2.11 (C5)
- net C36: now also LED2.6 (C6)
- net C37: now also LED2.2 (C7)
- net C38: now also LED2.1 (C8)
- net C41: now also LED5.4 (C1)
- net C42: now also LED5.14 (C2)
- net C43: now also LED5.13 (C3)
- net C44: now also LED5.7 (C4)
- net C45: now also LED5.11 (C5)
- net C46: now also LED5.6 (C6)
- net C47: now also LED5.2 (C7)
- net C48: now also LED5.1 (C8)
- net C51: now also LED3.4 (C1)
- net C52: now also LED3.14 (C2)
- net C53: now also LED3.13 (C3)
- net C54: now also LED3.7 (C4)
- net C55: now also LED3.11 (C5)
- net C56: now also LED3.6 (C6)
- net C57: now also LED3.2 (C7)
- net C58: now also LED3.1 (C8)
- net C61: now also LED6.4 (C1)
- net C62: now also LED6.14 (C2)
- net C63: now also LED6.13 (C3)
- net C64: now also LED6.7 (C4)
- net C65: now also LED6.11 (C5)
- net C66: now also LED6.6 (C6)
- net C67: now also LED6.2 (C7)
- net C68: now also LED6.1 (C8)
- net CLK: now also P3.2 (P2), P4.2 (P2), P9.1 (P1)
- net DIN: now also P1.2 (P2), P9.4 (P4)
- net GND: now also C1.2, C2.2, C3.2, C4.2, C5.2, C6.2, P1.1 (P1), P10.1 (P1), P10.2 (P2), P10.3 (P3), P10.4 (P4), P11.1 (P1), P11.2 (P2), P12.1 (P1), P12.2 (P2), P2.1 (P1), P5.1 (P1), P5.2 (P2), P5.3 (P3), P5.4 (P4), P6.1 (P1), P6.2 (P2), P6.3 (P3), P6.4 (P4)
- net LOAD: now also P3.1 (P1), P4.1 (P1), P9.3 (P3)
- net R11: now also LED1.8 (R1)
- net R12: now also LED1.3 (R2)
- net R13: now also LED1.9 (R3)
- net R14: now also LED1.5 (R4)
- net R15: now also LED1.16 (R5)
- net R16: now also LED1.10 (R6)
- net R17: now also LED1.15 (R7)
- net R18: now also LED1.12 (R8)
- net R21: now also LED4.8 (R1)
- net R22: now also LED4.3 (R2)
- net R23: now also LED4.9 (R3)
- net R24: now also LED4.5 (R4)
- net R25: now also LED4.16 (R5)
- net R26: now also LED4.10 (R6)
- net R27: now also LED4.15 (R7)
- net R28: now also LED4.12 (R8)
- net R31: now also LED2.8 (R1)
- net R32: now also LED2.3 (R2)
- net R33: now also LED2.9 (R3)
- net R34: now also LED2.5 (R4)
- net R35: now also LED2.16 (R5)
- net R36: now also LED2.10 (R6)
- net R37: now also LED2.15 (R7)
- net R38: now also LED2.12 (R8)
- net R41: now also LED5.8 (R1)
- net R42: now also LED5.3 (R2)
- net R43: now also LED5.9 (R3)
- net R44: now also LED5.5 (R4)
- net R45: now also LED5.16 (R5)
- net R46: now also LED5.10 (R6)
- net R47: now also LED5.15 (R7)
- net R48: now also LED5.12 (R8)
- net R51: now also LED3.8 (R1)
- net R52: now also LED3.3 (R2)
- net R53: now also LED3.9 (R3)
- net R54: now also LED3.5 (R4)
- net R55: now also LED3.16 (R5)
- net R56: now also LED3.10 (R6)
- net R57: now also LED3.15 (R7)
- net R58: now also LED3.12 (R8)
- net R61: now also LED6.8 (R1)
- net R62: now also LED6.3 (R2)
- net R63: now also LED6.9 (R3)
- net R64: now also LED6.5 (R4)
- net R65: now also LED6.16 (R5)
- net R66: now also LED6.10 (R6)
- net R67: now also LED6.15 (R7)
- net R68: now also LED6.12 (R8)
- net VCC: now also C1.1, C2.1, C3.1, C4.1, C5.1, C6.1, P11.3 (P3), P11.4 (P4), P12.3 (P3), P12.4 (P4), P7.1 (P1), P7.2 (P2), P7.3 (P3), P7.4 (P4), P8.1 (P1), P8.2 (P2), P8.3 (P3), P8.4 (P4), P9.2 (P2)
- net DOUT6: now reaches U6.24 (DOUT)
- net DOUT6: now also P2.2 (P2)
- no-connect marks 1 -> 0
Other:
- note added: "Connectors"
- note added: "Control"
- note added: "DIsplays"
- note added: "Power"
