File: Hardware/MatrixDisplay.kicad_pcb (KiCad board)
At the start: 2 copper layers, 64 x 96 mm, 36 parts, among them P1 CONN_01X02, P10 CONN_01X04, P11 CONN_01X04, P12 CONN_01X04, P2 CONN_01X02, P3 CONN_01X02, P4 CONN_01X02, P5 CONN_01X04, P6 CONN_01X04, P7 CONN_01X04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

Commit message: Gnerate gerber file
Routing:
- net VCC: vias 6 -> 12
- net GND: vias 8 -> 14
Other:
- rule pad_to_mask_clearance: 0.2 -> 0.2032
Changed lines of the file:
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@@
     (links 191)
     (no_connects 0)
-    (area 104.489467 31.6813 174.148534 135.7247)
+    (area 107.239999 35.929499 171.398001 132.091501)
     (thickness 1.6)
     (drawings 4)
-    (tracks 1092)
+    (tracks 1104)
     (zones 0)
     (modules 36)
@@
   )
   (page A4)
+  (title_block
+    (title MatrixDisplay)
+    (date 2016-08-08)
+    (rev 1)
+  )
   (layers
     (0 F.Cu signal)
@@
   )
   (setup
-    (last_trace_width 0.3048)
+    (last_trace_width 1.27)
     (user_trace_width 0.2032)
     (user_trace_width 0.254)
@@
     (pad_size 1.8 1.8)
     (pad_drill 1)
-    (pad_to_mask_clearance 0.2)
-    (aux_axis_origin 0 0)
+    (pad_to_mask_clearance 0.2032)
+    (aux_axis_origin 107.315 132.0165)
+    (grid_origin 107.315 132.0165)
     (visible_elements FFFFFF7F)
     (pcbplotparams
-      (layerselection 0x00030_80000001)
+      (layerselection 0x010f0_80000001)
       (usegerberextensions false)
       (excludeedgelayer true)
@@
       (psnegative false)
       (psa4output false)
-      (plotreference true)
-      (plotvalue true)
+      (plotreference false)
+      (plotvalue false)
       (plotinvisibletext false)
       (padsonsilk false)
-      (subtractmaskfromsilk false)
-      (outputformat 4)
+      (subtractmaskfromsilk true)
+      (outputformat 1)
       (mirror false)
       (drillshape 0)
@@
   (gr_line (start 171.323 132.0165) (end 171.323 36.0045) (angle 90) (layer Edge.Cuts) (width 0.15))
   (gr_line (start 107.315 132.0165) (end 171.323 132.0165) (angle 90) (layer Edge.Cuts) (width 0.15))
+  (via (at 164.846 70.8975) (size 1.2) (drill 0.7) (layers F.Cu B.Cu) (net 1))
+  (segment (start 165.1 69.2785) (end 164.846 69.0245) (width 1.27) (layer F.Cu) (net 1))
+  (via (at 164.846 69.0245) (size 1.2) (drill 0.7) (layers F.Cu B.Cu) (net 1))
+  (via (at 164.846 66.7385) (size 1.2) (drill 0.7) (layers F.Cu B.Cu) (net 1))
+  (segment (start 113.792 69.2785) (end 113.792 66.7385) (width 1.27) (layer F.Cu) (net 1))
+  (via (at 113.792 70.8975) (size 1.2) (drill 0.7) (layers F.Cu B.Cu) (net 1))
+  (via (at 113.792 69.2785) (size 1.2) (drill 0.7) (layers F.Cu B.Cu) (net 1))
+  (via (at 113.792 66.7385) (size 1.2) (drill 0.7) (layers F.Cu B.Cu) (net 1))
   (segment (start 124.521 93.9165) (end 124.521 83.6295) (width 0.508) (layer F.Cu) (net 1))
   (segment (start 124.521 83.6295) (end 124.521 65.4685) (width 0.508) (layer F.Cu) (net 1))
@@
   (segment (start 124.521 61.9125) (end 124.521 64.7065) (width 0.508) (layer F.Cu) (net 1))
   (via (at 124.521 64.7065) (size 0.6) (drill 0.4) (layers F.Cu B.Cu) (net 1))
-  (segment (start 113.792 69.2785) (end 113.792 66.7385) (width 1.27) (layer F.Cu) (net 1))
   (via (at 164.846 65.1195) (size 1.2) (drill 0.7) (layers F.Cu B.Cu) (net 1))
   (via (at 113.792 65.1195) (size 1.2) (drill 0.7) (layers F.Cu B.Cu) (net 1))
@@
   (segment (start 164.846 69.0245) (end 164.846 70.8975) (width 1.27) (layer F.Cu) (net 1))
   (segment (start 169.037 69.2785) (end 165.1 69.2785) (width 1.27) (layer F.Cu) (net 1))
-  (segment (start 165.1 69.2785) (end 164.846 69.0245) (width 1.27) (layer F.Cu) (net 1))
   (segment (start 169.037 64.1985) (end 165.767 64.1985) (width 1.27) (layer F.Cu) (net 1))
   (segment (start 165.767 64.1985) (end 164.846 65.1195) (width 1.27) (layer F.Cu) (net 1))
@@
   (segment (start 124.521 40.2615) (end 124.968 39.8145) (width 0.508) (layer F.Cu) (net 1))
   (segment (start 124.968 39.8145) (end 124.968 37.9095) (width 0.508) (layer F.Cu) (net 1))
+  (via (at 164.973 103.0605) (size 1.2) (drill 0.7) (layers F.Cu B.Cu) (net 2))
+  (via (at 164.973 101.2825) (size 1.2) (drill 0.7) (layers F.Cu B.Cu) (net 2))
+  (via (at 164.973 98.7425) (size 1.2) (drill 0.7) (layers F.Cu B.Cu) (net 2))
+  (via (at 113.665 103.0285) (size 1.2) (drill 0.7) (layers F.Cu B.Cu) (net 2))
+  (via (at 113.665 101.2825) (size 1.2) (drill 0.7) (layers F.Cu B.Cu) (net 2))
+  (via (at 113.665 98.7425) (size 1.2) (drill 0.7) (layers F.Cu B.Cu) (net 2))
   (segment (start 122.621 96.5835) (end 122.621 87.4395) (width 0.508) (layer F.Cu) (net 2))
   (segment (start 122.621 87.4395) (end 122.621 81.2165) (width 0.508) (layer F.Cu) (net 2))

Commit message: Change SOIC-24 package
Parts:
- U1, U2, U3, U4, U5, U6: footprint SMD_Packages:SOIC-24 -> SMD-my:SOIC-24-WIDTH
Routing:
- net C53: track 19.8 -> 17.0 mm
- net C43: track 19.8 -> 17.0 mm
- net C63: track 19.8 -> 17.0 mm
- net C62: track 20.5 -> 17.6 mm
- net C52: track 20.5 -> 17.8 mm
- net C33: track 19.6 -> 17.0 mm
- net C45: track 19.1 -> 16.5 mm
- net C42: track 20.3 -> 17.8 mm
- net C35: track 19.4 -> 17.0 mm
- net R21: track 27.4 -> 25.1 mm
- net C55: track 19.1 -> 16.8 mm
- net C65: track 19.1 -> 16.8 mm
- net R61: track 28.0 -> 25.9 mm
- net R51: track 27.5 -> 25.4 mm
- net R41: track 27.8 -> 25.7 mm
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Other:
- net class Default: trace_width 0.25 -> 0.2032
- rule via_min_size: 0.4 -> 0.508
